File: PCB Design/SPD PCB/SPD PCB.kicad_pcb (KiCad board)
At the start: 2 copper layers, 5 parts, among them Q1 2N2647, Q2 2N2647, U1 PN5321A3HN_C1xx, U2 ATmega328-P, U3 L293D

Commit message: c
Parts:
- removed U1: PN5321A3HN_C1xx, Package_DFN_QFN:HVQFN-40-1EP_6x6mm_P0.5mm_EP4.1x4.1mm
- added J1: Conn_01x06_Male, Connector_PinHeader_1.00mm:PinHeader_1x06_P1.00mm_Horizontal, F.Cu at (134.6, 91.4)
- added J2: Conn_01x02_Female, Connector_PinHeader_1.00mm:PinHeader_1x02_P1.00mm_Horizontal, F.Cu at (96.5, 78.7)
- added J3: Conn_01x02_Female, Connector_PinHeader_1.00mm:PinHeader_1x02_P1.00mm_Horizontal, F.Cu at (96.5, 114.3)
- added J4: Conn_01x05_Male, Connector_PinHeader_1.00mm:PinHeader_1x05_P1.00mm_Horizontal, F.Cu at (101.6, 132.1)
- added J5: Barrel_Jack, Connector_BarrelJack:BarrelJack_CLIFF_FC681465S_SMT_Horizontal, F.Cu at (142.2, 114.3)
- moved Q1 63.6 mm to (96.5, 91.4)
- moved Q2 58.5 mm to (96.5, 104.1)
- moved U3 37.8 mm to (115.6, 128.3)
Routing:
- net Earth: track 0.00 -> 172.6 mm
- net +5V: track 0.00 -> 139.4 mm
- net Net-(U2-Pad15): track 0.00 -> 41.9 mm
- net Net-(U2-Pad16): track 0.00 -> 34.7 mm
- net Net-(Q2-Pad2): track 0.00 -> 27.1 mm
- net Net-(U3-Pad11): track 0.00 -> 26.5 mm
- net Net-(U3-Pad14): track 0.00 -> 23.8 mm
- net Net-(U2-Pad17): track 0.00 -> 20.9 mm
- net Net-(Q1-Pad2): track 0.00 -> 20.9 mm
- net Net-(J4-Pad2): track 0.00 -> 18.1 mm
- net Net-(U2-Pad14): track 0.00 -> 17.4 mm
- net Net-(U3-Pad3): track 0.00 -> 15.3 mm
- net Net-(J2-Pad1): track 0.00 -> 14.1 mm
- net Net-(J1-Pad5): track 0.00 -> 12.4 mm
- net Net-(J1-Pad2): track 0.00 -> 12.4 mm
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Other:
- board outline added: 68.6 x 81.3 mm
