File: PCB Design/SPD PCB/SPD PCB.kicad_sch (KiCad schematic)
At the start: 3 parts

Commit message: touch ups on diagram
Parts:
- added M?: Stepper_Motor_unipolar_5pin, symbol Motor:Stepper_Motor_unipolar_5pin
- added M? (x2): Motor_DC, symbol Motor:Motor_DC
- added U?: ATmega328-P, Package_DIP:DIP-28_W7.62mm, symbol MCU_Microchip_ATmega:ATmega328-P
- added U?: L293D, Package_DIP:DIP-16_W7.62mm, symbol Driver_Motor:L293D
Connections:
- net Earth: now reaches Q?.1 (B2)
- net Earth: now also Q?.1 (B2), U?.12 (GND), U?.13 (GND), U?.4 (GND), U?.5 (GND), U?.8 (GND)
- net at Q?.2 (E): now also U?.2 (PD0)
- net at Q?.3 (B1): now also M?.2 (-) (x2)
- net at Q?.2 (E): now also U?.3 (PD1)
- new net: M?.2, U?.3 (1Y)
- new net: M?.3 (-), U?.6 (2Y)
- new net: M?.4, U?.11 (3Y)
- new net: M?.5, U?.14 (4Y)
- new net: U?.14 (PB0), U?.2 (1A)
- new net: U?.15 (PB1), U?.7 (2A)
- new net: U?.10 (3A), U?.16 (PB2)
- new net: U?.15 (4A), U?.17 (PB3)
- new net +5V: M?.1, M?.1 (+), M?.1 (+), U?.1 (EN1,2), U?.16 (VCC1), U?.8 (VCC2), U?.9 (EN3,4)
Other:
- moved on the sheet: Q?, U?

Commit message: d
Parts:
- gave numbers to parts that had none: 8
Connections:
- net at U2.23 (PC0): now also U1.30 (SCK/P72)
- net at U2.24 (PC1): now also U1.29 (MISO/P71)
- net at U2.25 (PC2): now also U1.28 (MOSI/SDA/HSU_TX)
- net at U2.26 (PC3): now also U1.27 (NSS/P50_SCL/HSU_RX)
Other:
- moved on the sheet: U1
Changed lines of the file:
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@@
+    (stroke (width 0) (type default) (color 0 0 0 0))
+  )
+  (wire (pts (xy 64.77 114.3) (xy 64.77 73.66))
     (stroke (width 0) (type default) (color 0 0 0 0))
   )
@@
     (stroke (width 0) (type default) (color 0 0 0 0))
   )
+  (wire (pts (xy 62.23 114.3) (xy 62.23 76.2))
+    (stroke (width 0) (type default) (color 0 0 0 0))
+  )
   (wire (pts (xy 259.08 109.22) (xy 259.08 120.65))
     (stroke (width 0) (type default) (color 0 0 0 0))
@@
     (stroke (width 0) (type default) (color 0 0 0 0))
   )
+  (wire (pts (xy 59.69 114.3) (xy 59.69 78.74))
+    (stroke (width 0) (type default) (color 0 0 0 0))
+  )
   (wire (pts (xy 123.19 36.83) (xy 144.78 36.83))
     (stroke (width 0) (type default) (color 0 0 0 0))
@@
     (stroke (width 0) (type default) (color 0 0 0 0))
   )
+  (wire (pts (xy 64.77 73.66) (xy 92.71 73.66))
+    (stroke (width 0) (type default) (color 0 0 0 0))
+  )
   (wire (pts (xy 172.72 20.32) (xy 167.64 20.32))
     (stroke (width 0) (type default) (color 0 0 0 0))
@@
     (stroke (width 0) (type default) (color 0 0 0 0))
   )
+  (wire (pts (xy 67.31 71.12) (xy 92.71 71.12))
+    (stroke (width 0) (type default) (color 0 0 0 0))
+  )
   (wire (pts (xy 185.42 121.92) (xy 185.42 88.9))
     (stroke (width 0) (type default) (color 0 0 0 0))
@@
     (stroke (width 0) (type default) (color 0 0 0 0))
   )
+  (wire (pts (xy 59.69 78.74) (xy 92.71 78.74))
+    (stroke (width 0) (type default) (color 0 0 0 0))
+  )
   (wire (pts (xy 172.72 76.2) (xy 172.72 88.9))
     (stroke (width 0) (type default) (color 0 0 0 0))
@@
     (stroke (width 0) (type default) (color 0 0 0 0))
   )
+  (wire (pts (xy 62.23 76.2) (xy 92.71 76.2))
+    (stroke (width 0) (type default) (color 0 0 0 0))
+  )
   (wire (pts (xy 172.72 88.9) (xy 175.26 88.9))
     (stroke (width 0) (type default) (color 0 0 0 0))
@@
   )
   (wire (pts (xy 215.9 36.83) (xy 215.9 43.18))
+    (stroke (width 0) (type default) (color 0 0 0 0))
+  )
+  (wire (pts (xy 67.31 114.3) (xy 67.31 71.12))
     (stroke (width 0) (type default) (color 0 0 0 0))
   )
@@
   (symbol (lib_id "power:+5V") (at 156.21 20.32 0) (unit 1)
     (in_bom yes) (on_board yes) (fields_autoplaced)
-    (property "Reference" "#PWR?" (id 0) (at 156.21 24.13 0)
+    (property "Reference" "#PWR0103" (id 0) (at 156.21 24.13 0)
       (effects (font (size 1.27 1.27)) hide)
     )
@@
   (symbol (lib_id "Motor:Stepper_Motor_unipolar_5pin") (at 213.36 50.8 0) (unit 1)
     (in_bom yes) (on_board yes) (fields_autoplaced)
-    (property "Reference" "M?" (id 0) (at 218.44 48.552 0)
+    (property "Reference" "M1" (id 0) (at 218.44 48.552 0)
       (effects (font (size 1.27 1.27)) (justify left))
     )
@@
   (symbol (lib_id "power:Earth") (at 177.8 88.9 0) (unit 1)
     (in_bom yes) (on_board yes) (fields_autoplaced)
-    (property "Reference" "#PWR?" (id 0) (at 177.8 95.25 0)
+    (property "Reference" "#PWR0102" (id 0) (at 177.8 95.25 0)
       (effects (font (size 1.27 1.27)) hide)
     )
@@
   (symbol (lib_id "Motor:Motor_DC") (at 231.14 128.27 180) (unit 1)
     (in_bom yes) (on_board yes) (fields_autoplaced)
-    (property "Reference" "M?" (id 0) (at 236.22 124.4599 0)
+    (property "Reference" "M3" (id 0) (at 236.22 124.4599 0)
       (effects (font (size 1.27 1.27)) (justify right))
     )
@@
   (symbol (lib_id "Transistor_BJT:2N2647") (at 195.58 102.87 0) (unit 1)
     (in_bom yes) (on_board yes) (fields_autoplaced)
-    (property "Reference" "Q?" (id 0) (at 200.66 101.5999 0)
+    (property "Reference" "Q1" (id 0) (at 200.66 101.5999 0)
       (effects (font (size 1.27 1.27)) (justify left))
     )
@@
   (symbol (lib_id "Transistor_BJT:2N2647") (at 195.58 127 0) (unit 1)
     (in_bom yes) (on_board yes) (fields_autoplaced)
-    (property "Reference" "Q?" (id 0) (at 200.66 125.7299 0)
+    (property "Reference" "Q2" (id 0) (at 200.66 125.7299 0)
       (effects (font (size 1.27 1.27)) (justify left))
     )
@@
   (symbol (lib_id "MCU_Microchip_ATmega:ATmega328-P") (at 107.95 67.31 0) (unit 1)
     (in_bom yes) (on_board yes) (fields_autoplaced)
-    (property "Reference" "U?" (id 0) (at 86.36 32.4993 0))
+    (property "Reference" "U2" (id 0) (at 86.36 32.4993 0))
     (property "Value" "ATmega328-P" (id 1) (at 86.36 35.0393 0))
     (property "Footprint" "Package_DIP:DIP-28_W7.62mm" (id 2) (at 107.95 71.12 0)
@@
   (symbol (lib_id "Driver_Motor:L293D") (at 170.18 55.88 0) (unit 1)
     (in_bom yes) (on_board yes) (fields_autoplaced)
-    (property "Reference" "U?" (id 0) (at 174.7394 27.94 0)
+    (property "Reference" "U3" (id 0) (at 174.7394 27.94 0)
       (effects (font (size 1.27 1.27)) (justify left))
     )
@@
   (symbol (lib_id "power:+5V") (at 274.32 120.65 270) (unit 1)
     (in_bom yes) (on_board yes) (fields_autoplaced)
-    (property "Reference" "#PWR?" (id 0) (at 270.51 120.65 0)
+    (property "Reference" "#PWR0101" (id 0) (at 270.51 120.65 0)
       (effects (font (size 1.27 1.27)) hide)
     )
@@
     (pin "1")
   )
-  (symbol (lib_id "RF_NFC:PN5321A3HN_C1xx") (at 49.53 146.05 0) (unit 1)
+  (symbol (lib_id "RF_NFC:PN5321A3HN_C1xx") (at 54.61 134.62 270) (unit 1)
     (in_bom yes) (on_board yes)
-    (property "Reference" "U?" (id 0) (at 56.6294 110.49 0)
-      (effects (font (size 1.27 1.27)) (justify left))
-    )
-    (property "Value" "PN5321A3HN_C1xx" (id 1) (at 56.6294 113.03 0)
-      (effects (font (size 1.27 1.27)) (justify left))
-    )
-    (property "Footprint" "Package_DFN_QFN:HVQFN-40-1EP_6x6mm_P0.5mm_EP4.1x4.1mm" (id 2) (at 87.63 177.8 0)
-      (effects (font (size 1.27 1.27)) hide)
-    )
-    (property "Datasheet" "https://www.nxp.com/docs/en/nxp/data-sheets/PN532_C1.pdf" (id 3) (at 49.53 140.97 0)
+    (property "Reference" "U1" (id 0) (at 90.17 141.7194 0)
+      (effects (font (size 1.27 1.27)) (justify left))
+    )
+    (property "Value" "PN5321A3HN_C1xx" (id 1) (at 87.63 141.7194 0)
+      (effects (font (size 1.27 1.27)) (justify left))
+    )
+    (property "Footprint" "Package_DFN_QFN:HVQFN-40-1EP_6x6mm_P0.5mm_EP4.1x4.1mm" (id 2) (at 22.86 172.72 0)
+      (effects (font (size 1.27 1.27)) hide)
+    )
+    (property "Datasheet" "https://www.nxp.com/docs/en/nxp/data-sheets/PN532_C1.pdf" (id 3) (at 59.69 134.62 0)
       (effects (font (size 1.27 1.27)) hide)
     )
@@
   (symbol (lib_id "Motor:Motor_DC") (at 231.14 104.14 180) (unit 1)
     (in_bom yes) (on_board yes) (fields_autoplaced)
-    (property "Reference" "M?" (id 0) (at 236.22 100.3299 0)
+    (property "Reference" "M2" (id 0) (at 236.22 100.3299 0)
       (effects (font (size 1.27 1.27)) (justify right))
     )
@@
   )
   (symbol_instances
+    (path "/9dde75c5-cd76-416e-b923-f49594bcc604"
+      (reference "#PWR0101") (unit 1) (value "+5V") (footprint "")
+    )
+    (path "/3e692965-d700-4c46-a3a6-40e4a3addd69"
+      (reference "#PWR0102") (unit 1) (value "Earth") (footprint "")
+    )
     (path "/00a9889f-f796-401f-b802-1f8d656eabfa"
-      (reference "#PWR?") (unit 1) (value "+5V") (footprint "")
-    )
-    (path "/3e692965-d700-4c46-a3a6-40e4a3addd69"
-      (reference "#PWR?") (unit 1) (value "Earth") (footprint "")
-    )
-    (path "/9dde75c5-cd76-416e-b923-f49594bcc604"
-      (reference "#PWR?") (unit 1) (value "+5V") (footprint "")
+      (reference "#PWR0103") (unit 1) (value "+5V") (footprint "")
     )
     (path "/010c43a2-732c-48b0-bbc7-9b5dac471893"
-      (reference "M?") (unit 1) (value "Stepper_Motor_unipolar_5pin") (footprint "")
+      (reference "M1") (unit 1) (value "Stepper_Motor_unipolar_5pin") (footprint "")
+    )
+    (path "/de7623af-3a24-42bc-add7-afe601da191d"
+      (reference "M2") (unit 1) (value "Motor_DC") (footprint "")
     )
     (path "/486d0cbe-4acc-44ba-be23-b0e9a26ebe54"
-      (reference "M?") (unit 1) (value "Motor_DC") (footprint "")
-    )
-    (path "/de7623af-3a24-42bc-add7-afe601da191d"
-      (reference "M?") (unit 1) (value "Motor_DC") (footprint "")
+      (reference "M3") (unit 1) (value "Motor_DC") (footprint "")
     )
     (path "/614cdb19-2c65-4827-8b39-3188640573dd"
-      (reference "Q?") (unit 1) (value "2N2647") (footprint "Package_TO_SOT_THT:TO-18-3")
+      (reference "Q1") (unit 1) (value "2N2647") (footprint "Package_TO_SOT_THT:TO-18-3")
     )
     (path "/635a8034-da7e-4fe0-9f67-ae1afad1e2cd"
-      (reference "Q?") (unit 1) (value "2N2647") (footprint "Package_TO_SOT_THT:TO-18-3")
+      (reference "Q2") (unit 1) (value "2N2647") (footprint "Package_TO_SOT_THT:TO-18-3")
+    )
+    (path "/b199093d-fc35-4a57-84d4-9203d9dc1821"
+      (reference "U1") (unit 1) (value "PN5321A3HN_C1xx") (footprint "Package_DFN_QFN:HVQFN-40-1EP_6x6mm_P0.5mm_EP4.1x4.1mm")
     )
     (path "/67b819b7-12c7-4dd7-bd3a-61ec6664e433"
-      (reference "U?") (unit 1) (value "ATmega328-P") (footprint "Package_DIP:DIP-28_W7.62mm")
+      (reference "U2") (unit 1) (value "ATmega328-P") (footprint "Package_DIP:DIP-28_W7.62mm")
     )
     (path "/77e25307-4c6e-44db-8aa1-41dfa691957f"
-      (reference "U?") (unit 1) (value "L293D") (footprint "Package_DIP:DIP-16_W7.62mm")
-    )
-    (path "/b199093d-fc35-4a57-84d4-9203d9dc1821"
-      (reference "U?") (unit 1) (value "PN5321A3HN_C1xx") (footprint "Package_DFN_QFN:HVQFN-40-1EP_6x6mm_P0.5mm_EP4.1x4.1mm")
-    )
-  )
+      (reference "U3") (unit 1) (value "L293D") (footprint "Package_DIP:DIP-16_W7.62mm")
+    )
+  )

Commit message: d
Parts:
- added J1: Conn_01x06_Male, symbol Connector:Conn_01x06_Male
- added J2, J?: Conn_01x02_Female, symbol Connector:Conn_01x02_Female
- added J?: Conn_01x05_Male, symbol Connector:Conn_01x05_Male
Connections:
- net +5V: now also J?.1 (Pin_1); no longer M1.1, M2.1 (+), M3.1 (+)
- net at M1.2: no longer U3.3 (1Y)
- net at M1.3 (-): no longer U3.6 (2Y)
- net at M1.4: no longer U3.11 (3Y)
- net at M1.5: no longer U3.14 (4Y)
- net at M3.2 (-): no longer Q2.3 (B1)
- net at Q1.3 (B1): now also J2.1 (Pin_1); no longer M2.2 (-)
- net at U2.23 (PC0): now also J1.5 (Pin_5); no longer U1.30 (SCK/P72)
- net at U2.24 (PC1): now also J1.4 (Pin_4); no longer U1.29 (MISO/P71)
- net at U2.25 (PC2): now also J1.3 (Pin_3); no longer U1.28 (MOSI/SDA/HSU_TX)
- net at U2.26 (PC3): now also J1.2 (Pin_2); no longer U1.27 (NSS/P50_SCL/HSU_RX)
- new net: J?.1 (Pin_1), Q2.3 (B1)
- new net: J?.4 (Pin_4), U3.11 (3Y)
- new net: J?.5 (Pin_5), U3.14 (4Y)
- new net: J?.3 (Pin_3), U3.3 (1Y)
- new net: J?.2 (Pin_2), U3.6 (2Y)
Other:
- moved on the sheet: M1

Commit message: c
Parts:
- added J5: Barrel_Jack, Connector_BarrelJack:BarrelJack_CLIFF_FC681465S_SMT_Horizontal, symbol Connector:Barrel_Jack
- J1: footprint (none) -> Connector_PinHeader_1.00mm:PinHeader_1x06_P1.00mm_Horizontal
- J2, M1: footprint (none) -> Connector_PinHeader_1.00mm:PinHeader_1x02_P1.00mm_Horizontal
- J3: renamed from J?; footprint (none) -> Connector_PinHeader_1.00mm:PinHeader_1x02_P1.00mm_Horizontal
- J4: renamed from J?; footprint (none) -> Connector_PinHeader_1.00mm:PinHeader_1x05_P1.00mm_Horizontal
Connections:
- net +5V: now also J2.2 (Pin_2), J3.2 (Pin_2), J5.1; no longer J4.1 (Pin_1)
- net Earth: now also J1.1 (Pin_1), J4.1 (Pin_1), J5.2
